File: homeAutomationPCB/esp32_wk40/esp32_wk40.sch (KiCad schematic (older format))
At the start: 55 parts, among them J1 Conn_01x05_Male, J2 Conn_01x02_Male, J3 Screw_Terminal_01x02, J4 Screw_Terminal_01x02, J5 Screw_Terminal_01x02, J6 Screw_Terminal_01x02, J7 Screw_Terminal_01x05, J8 Screw_Terminal_01x02, J9 Conn_01x05_Male, Q3 BC547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

Commit message: Added CHANGELOG.rst
Parts:
- U10, U11, U8, U9: symbol new_components:RZ03-1A3-D005 -> esp32_wk40-rescue:RZ03-1A3-D005-new_components
Connections:
- new net: J7.5 (Pin_5), U10.~ (A2), U11.~ (A2), U8.~ (A2), U9.~ (A2)
Changed lines of the file:
@@
 	1380 1730 1380 1670
 $Comp
-L new_components:RZ03-1A3-D005 U10
+L esp32_wk40-rescue:RZ03-1A3-D005-new_components U10
 U 1 1 5F6996B7
 P 14670 850
@@
 $EndComp
 $Comp
-L new_components:RZ03-1A3-D005 U9
+L esp32_wk40-rescue:RZ03-1A3-D005-new_components U9
 U 1 1 5FC74058
 P 14580 2560
@@
 $EndComp
 $Comp
-L new_components:RZ03-1A3-D005 U8
+L esp32_wk40-rescue:RZ03-1A3-D005-new_components U8
 U 1 1 5FC7F8C2
 P 14490 4240
@@
 $EndComp
 $Comp
-L new_components:RZ03-1A3-D005 U11
+L esp32_wk40-rescue:RZ03-1A3-D005-new_components U11
 U 1 1 5FC8BC04
 P 14440 6010
